Commit message: spoj gazebo&rviz radi na pola

File: xarm_ros_nongit/xarm_description/urdf/xarm5.transmission.xacro (robot description, xacro)
@@ -1,5 +1,5 @@
 <?xml version="1.0"?>
 <robot xmlns:xacro="http://ros.org/wiki/xacro">
-  <xacro:macro name="xarm5_transmission"
+ <xacro:macro name="xarm5_transmission"
     params="prefix hard_interface:=EffortJointInterface reduction:=100">
     <transmission name="${prefix}tran1">
