Commit message: Phantomx_arm napravljen rviz u spoju s moveit (ne radi y-os na robotu)

File: phantomx_arm/phantomx_reactor_arm_description/urdf/phantomx_reactor_arm_wrist.urdf.xacro (robot description, xacro)
@@ -10,4 +10,10 @@
 			</geometry>
 		</visual>
+		<collision>
+			<origin xyz="0 0 0" rpy="0 0 0"/>
+			<geometry>
+				<box size="0.001 0.001 0.001" />
+			</geometry>
+		</collision>
 	</link>
 	<xacro:phantomx_reactor_wrist prefix="" parent="base_footprint">

File: phantomx_arm/phantomx_reactor_arm_description/urdf/phantomx_reactor_wrist.urdf.xacro (robot description, xacro)
@@ -1,4 +1,4 @@
 <?xml version="1.0"?>
-<robot name="phantomx_reactor" xmlns:xacro="http://www.ros.org/wiki/xacro">
+<robot name="phantomx_reactor" xmlns:xacro="http://ros.org/wiki/xacro">
 	<xacro:property name="PI" value="3.141593"/>
 	<xacro:property name="shoulder_yaw_joint_upper_limit" value="${PI}"/>
